File: Panel4/pcb/Maker Faire Machine Panel4 (Electron).sch (EAGLE design)
At the start: 26 parts, among them IC1 TJA1049

Commit message: First version of panel 4 PCB done
Parts:
- JP1: device panel4:M10X2MOLEX_MX150 -> panel4:M10X2_MMOLEX_MX150; PARTNO (none) -> 348302001
- JP2: DNP (none) -> T
- U$2: value SPARK_LOGO.. -> SPARK_LOGOSILK; device Spark:SPARK_LOGO.. -> Spark:SPARK_LOGOSILK; BOM (none) -> EXCLUDE
Other:
- moved on the sheet: C3, IC1
